File: Harpe ruches/Fichier Kicad/Harpe_ESP32/Harpe_ESP32.kicad_pcb (KiCad board)
At the start: 2 copper layers, 69.3 x 100 mm, 66 parts, among them J1 Conn_01x04, J10 Screw_Terminal_01x02, J13 USB_C_Receptacle_USB2.0 USB41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, J2 Conn_01x02_MountingPin, J3 Conn_01x02_MountingPin, J4 Conn_01x02_MountingPin, J5 Conn_01x02_MountingPin, J6 Conn_01x02_MountingPin, J7 Conn_01x04, J8 Conn_01x02_MountingPin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

Commit message: Update
Other:
- board text removed: "- Bat +"

Commit message: Update PCB
Parts:
- added R8: 10K, Resistor_SMD:R_0603_1608Metric, F.Cu at (117.6, 112.2)
- added SW2: SW_Push, Empreintes:PTS636SL43SMTRLFS, F.Cu at (121.2, 109.6)
- moved FID1 6.78 mm to (129.9, 79.9)
- moved D15 4.01 mm to (122.2, 112.2), turned to 90 degrees
Routing:
- net Vout5V: track 24.0 -> 21.2 mm
- net +3V3: track 130.7 -> 133.1 mm
- net I012: track 0.00 -> 1.97 mm
- net GND: track 23.4 -> 23.3 mm, vias 164 -> 165
Other:
- board text added: "- Bat +"

Commit message: Update PCB
Parts:
- added J11: Conn_01x04, Empreintes:1190297, F.Cu at (117.9, 154.1)
- added J9: Conn_01x02, Connector_JST:JST_PH_B2B-PH-K_1x02_P2.00mm_Vertical, F.Cu at (129.6, 89.6)
- J10: value Screw_Terminal_01x02 -> Conn_01x02; footprint Empreintes:1190297 -> Connector_JST:JST_PH_B2B-PH-K_1x02_P2.00mm_Vertical
- J2, J3, J4, J5, J6, J8: value Conn_01x02_MountingPin -> Conn_01x04
- moved J10 60.0 mm to (129.7, 95.3)
- moved FID3 5.66 mm to (161.0, 79.4)
- moved G*** 2.77 mm to (131.0, 154.0)
- moved R3 1.64 mm to (132.7, 101.3)
- moved R29 1.47 mm to (120.9, 113.2)
- moved D15 1.30 mm to (122.9, 113.2)
- moved G*** 1.11 mm to (124.7, 130.0)
- moved SW2 0.52 mm to (121.2, 109.1)
- moved FID1 0.46 mm to (130.1, 79.5)
Connections:
- J10 pad 1: GND -> RST_EN
- J10 pad 2: (no net) -> GND
- J2 pad 2: (no net) -> Net-(J2-Pin_1)
- J2 pad 4: (no net) -> GND
- J3 pad 2: (no net) -> Net-(J3-Pin_1)
- J3 pad 4: (no net) -> GND
- J4 pad 2: (no net) -> Net-(J4-Pin_1)
- J4 pad 4: (no net) -> GND
- J5 pad 2: (no net) -> Net-(J5-Pin_1)
- J5 pad 4: (no net) -> GND
- J6 pad 2: (no net) -> Net-(J6-Pin_1)
- J6 pad 4: (no net) -> GND
- J8 pad 2: (no net) -> Net-(J8-Pin_1)
- J8 pad 4: (no net) -> GND
- R8 pad 1: I012 -> I027
- SW2 pad 1: I012 -> I027
- U1 pad 12: unconnected-(U1-IO27-Pad12) -> I027
- U1 pad 37: unconnected-(U1-IO23-Pad37) -> I023
- U4 pad 3: Net-(J4-Pin_1) -> unconnected-(U4-Pad3)
Routing:
- net I027: track 0.00 -> 59.9 mm, vias 0 -> 3
- net RST_EN: track 38.1 -> 54.2 mm
- net Net-(J5-Pin_1): track 6.74 -> 14.9 mm
- net Net-(J4-Pin_1): track 6.77 -> 15.0 mm
- net Net-(J8-Pin_1): track 6.75 -> 15.0 mm
- net Net-(J6-Pin_1): track 6.56 -> 14.8 mm
- net Net-(J3-Pin_1): track 6.77 -> 15.0 mm
- net Net-(J2-Pin_1): track 6.74 -> 14.9 mm
- net VBAT: track 198.2 -> 201.1 mm
- net IO18: track 14.9 -> 17.5 mm
- net GND: track 23.3 -> 25.4 mm, vias 165 -> 164
- net I012: track 1.97 -> 0.00 mm
- net Net-(JP21-Pad2): track 2.94 -> 4.72 mm
- net Net-(R3-Pad1): track 2.88 -> 3.93 mm
Other:
- board text added: "Harpe n°1"
- board text added: "Harpe n°2"
- board text added: "Harpe n°3"
- board text added: "Harpe n°4"
- board text added: "Harpe n°5"
- board text added: "Harpe n°6"
- board text added: "SHT41 Capteur d'humidité"
- board text added: "VEML7700 Capteur de luminosité"
- board text added: "WIFI"
- board text removed: "SHT41 Humidity sensor"
- board text removed: "VEML7700 Luminosity sensor"

Commit message: update
Parts:
- removed FID4: Fiducial, Fiducial:Fiducial_1.5mm_Mask3mm
- J11, J2, J3, J4, J5, J6, J8: footprint Empreintes:1190297 -> Empreintes:1862411
- moved J4 11.0 mm to (161.7, 118.2)
- moved J5 11.0 mm to (161.7, 131.7)
- moved J2 11.0 mm to (161.7, 91.2)
- moved J8 11.0 mm to (161.7, 158.8)
- moved J3 11.0 mm to (161.7, 104.7)
- moved J6 11.0 mm to (161.7, 145.3)
- moved J11 10.8 mm to (118.4, 164.8)
- moved PS1 5.38 mm to (123.4, 146.0)
- moved G*** 4.38 mm to (144.9, 162.4)
- moved G*** 4.04 mm to (121.8, 132.8)
Connections:
- U4 pad 3: unconnected-(U4-Pad3) -> Net-(J4-Pin_1)
Routing:
- net VBAT: track 201.1 -> 229.5 mm
- net Net-(J3-Pin_1): track 15.0 -> 22.8 mm
- net Net-(J2-Pin_1): track 14.9 -> 22.8 mm
- net Vout5V: track 21.2 -> 26.6 mm
- net Net-(J8-Pin_1): track 15.0 -> 17.8 mm
- net Net-(J6-Pin_1): track 14.8 -> 17.6 mm
- net Net-(J4-Pin_1): track 15.0 -> 17.8 mm
- net Net-(J5-Pin_1): track 14.9 -> 17.7 mm
Other:
- board text added: "Ratamuse"
- board text removed: "- Bat +"
