File: Harpe ruches/Fichier Kicad/Harpe_ESP32/Harpe_ESP32.kicad_pcb (KiCad board)
At the start: 2 copper layers, 69.3 x 100 mm, 69 parts, among them J1 Conn_01x04, J10 Conn_01x02, J11 Conn_01x04, J13 USB_C_Receptacle_USB2.0 USB41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, J2 Conn_01x04, J3 Conn_01x04, J4 Conn_01x04, J5 Conn_01x04, J6 Conn_01x04, J7 Conn_01x04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

Commit message: update
Parts:
- added FID4: Fiducial, Fiducial:Fiducial_1.5mm_Mask3mm, F.Cu at (181.8, 88.3)
- U2, U3, U4, U5, U6, U7: value PC817 -> G3VM-61VY2; footprint Empreintes:SOP254P960X420-4N -> Empreintes:SOP254P700X230-4N
- moved REF** 3.89 mm to (107.2, 89.1)
- moved REF** 3.65 mm to (100.8, 88.9)
- moved R3 1.58 mm to (132.8, 99.7)
- moved G*** 1.37 mm to (127.8, 103.1)
- moved U2 0.29 mm to (140.4, 87.5)
- moved U3 0.28 mm to (140.3, 101.0)
- moved U5 0.20 mm to (140.4, 128.0)
- moved U4 0.19 mm to (140.4, 114.5)
- moved U7 0.16 mm to (140.5, 155.1)
- moved U6 0.13 mm to (140.7, 141.5)
Routing:
- net VBAT: track 229.5 -> 226.6 mm
- net Net-(J2-Pin_1): track 22.8 -> 24.1 mm
- net Net-(J5-Pin_1): track 17.7 -> 19.0 mm
- net Net-(J4-Pin_1): track 17.8 -> 19.0 mm
- net Net-(J8-Pin_1): track 17.8 -> 19.0 mm
- net Net-(J6-Pin_1): track 17.6 -> 18.8 mm
- net Net-(J3-Pin_1): track 22.8 -> 23.9 mm
- net Net-(R6-Pad1): track 3.07 -> 4.00 mm
- net Net-(R7-Pad1): track 2.69 -> 3.59 mm
- net Net-(R5-Pad1): track 3.73 -> 4.59 mm
- net Net-(R4-Pad1): track 3.07 -> 3.92 mm
- net Net-(R2-Pad1): track 2.88 -> 3.66 mm
- net IO18: track 17.5 -> 17.0 mm

Commit message: pcb updated
Parts:
- removed FID4: Fiducial, Fiducial:Fiducial_1.5mm_Mask3mm
Routing:
- net VBAT: track 226.6 -> 237.0 mm
Changed lines of the file:
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@@
     )
   )
-  (footprint "Fiducial:Fiducial_1.5mm_Mask3mm" (layer "F.Cu")
-    (at 181.775 88.255)
-    (descr "Circular Fiducial, 1.5mm bare copper, 3mm soldermask opening")
-    (tags "fiducial")
-    (property "Sheetfile" "Harpe_ESP32.kicad_sch")
-    (property "Sheetname" "")
-    (property "ki_description" "Fiducial Marker")
-    (property "ki_keywords" "fiducial marker")
-    (attr smd)
-    (fp_text reference "FID4" (at 0 -2.4765) (layer "F.SilkS")
-        (effects (font (size 1 1) (thickness 0.15)))
-    )
-    (fp_text value "Fiducial" (at 0 2.6035) (layer "F.Fab")
-        (effects (font (size 1 1) (thickness 0.15)))
-    )
-    (fp_text user "${REFERENCE}" (at 0 0) (layer "F.Fab")
-        (effects (font (size 0.4 0.4) (thickness 0.06)))
-    )
-    (fp_circle (center 0 0) (end 1.75 0)
-      (stroke (width 0.05) (type solid)) (fill none) (layer "F.CrtYd"))
-    (fp_circle (center 0 0) (end 1.5 0)
-      (stroke (width 0.1) (type solid)) (fill none) (layer "F.Fab"))
-    (pad "" smd circle (at 0 0) (size 1.5 1.5) (layers "F.Cu" "F.Mask")
-      (solder_mask_margin 0.75) (clearance 0.75))
-  )
   (footprint "Empreintes:SOP254P700X230-4N" (layer "F.Cu")
     (at 140.42 114.52)
@@
   (segment (start 110.4425 107.91) (end 109.75 107.91) (width 0.2) (layer "F.Cu") (net 1))
   (via (at 164.86 128.17) (size 0.65) (drill 0.3) (layers "F.Cu" "B.Cu") (net 1))
-  (via (at 136.57 144.36) (size 0.65) (drill 0.3) (layers "F.Cu" "B.Cu") (free) (net 1))
+  (via (at 135.9 142.8) (size 0.65) (drill 0.3) (layers "F.Cu" "B.Cu") (free) (net 1))
   (via (at 121.44 107.75) (size 0.65) (drill 0.3) (layers "F.Cu" "B.Cu") (net 1))
-  (via (at 136.3 117.31) (size 0.65) (drill 0.3) (layers "F.Cu" "B.Cu") (free) (net 1))
+  (via (at 135.6 115.81) (size 0.65) (drill 0.3) (layers "F.Cu" "B.Cu") (free) (net 1))
   (via (at 100.74 89.56) (size 0.65) (drill 0.3) (layers "F.Cu" "B.Cu") (net 1))
   (via (at 106.52 116.46) (size 0.65) (drill 0.3) (layers "F.Cu" "B.Cu") (net 1))
@@
   (via (at 108.78 90.23) (size 0.65) (drill 0.3) (layers "F.Cu" "B.Cu") (net 1))
   (via (at 164.86 75.45) (size 0.65) (drill 0.3) (layers "F.Cu" "B.Cu") (free) (net 1))
-  (via (at 136.37 103.83) (size 0.65) (drill 0.3) (layers "F.Cu" "B.Cu") (free) (net 1))
+  (via (at 135.56 102.21) (size 0.65) (drill 0.3) (layers "F.Cu" "B.Cu") (free) (net 1))
   (via (at 164.86 135.92) (size 0.65) (drill 0.3) (layers "F.Cu" "B.Cu") (net 1))
   (via (at 109.69 87.46) (size 0.65) (drill 0.3) (layers "F.Cu" "B.Cu") (net 1))
@@
   (via (at 164.86 92.95) (size 0.65) (drill 0.3) (layers "F.Cu" "B.Cu") (net 1))
   (via (at 105.86 167.75) (size 0.65) (drill 0.3) (layers "F.Cu" "B.Cu") (net 1))
-  (via (at 136.41 90.27) (size 0.65) (drill 0.3) (layers "F.Cu" "B.Cu") (free) (net 1))
+  (via (at 135.53 88.75) (size 0.65) (drill 0.3) (layers "F.Cu" "B.Cu") (free) (net 1))
   (via (at 139.08 70.71) (size 0.65) (drill 0.3) (layers "F.Cu" "B.Cu") (free) (net 1))
   (via (at 135.86 167.75) (size 0.65) (drill 0.3) (layers "F.Cu" "B.Cu") (net 1))
@@
   (via (at 98.1 81.59) (size 0.65) (drill 0.3) (layers "F.Cu" "B.Cu") (net 1))
   (via (at 164.86 82.95) (size 0.65) (drill 0.3) (layers "F.Cu" "B.Cu") (net 1))
-  (via (at 136.39 130.92) (size 0.65) (drill 0.3) (layers "F.Cu" "B.Cu") (free) (net 1))
-  (via (at 136.34 157.86) (size 0.65) (drill 0.3) (layers "F.Cu" "B.Cu") (free) (net 1))
+  (via (at 135.63 129.31) (size 0.65) (drill 0.3) (layers "F.Cu" "B.Cu") (free) (net 1))
+  (via (at 135.62 156.31) (size 0.65) (drill 0.3) (layers "F.Cu" "B.Cu") (free) (net 1))
   (via (at 98.07 128.22) (size 0.65) (drill 0.3) (layers "F.Cu" "B.Cu") (net 1))
   (via (at 125.32 102.8) (size 0.65) (drill 0.3) (layers "F.Cu" "B.Cu") (net 1))
@@
   (segment (start 147 99.69) (end 145.13 99.69) (width 1) (layer "F.Cu") (net 37))
   (segment (start 143.98 140.25) (end 145.51 140.25) (width 0.6) (layer "F.Cu") (net 37))
-  (segment (start 159.2 163.01) (end 159.2 83.79) (width 1) (layer "F.Cu") (net 37))
+  (segment (start 149.1 86.23) (end 145.25 86.23) (width 1) (layer "F.Cu") (net 37))
   (segment (start 145.15 113.25) (end 145.19 113.29) (width 0.5) (layer "F.Cu") (net 37))
+  (segment (start 123.41 146.035) (end 123.41 164.82) (width 1) (layer "F.Cu") (net 37))
   (segment (start 145.12 99.68) (end 145.13 99.69) (width 0.6) (layer "F.Cu") (net 37))
   (segment (start 158.97 150.58) (end 159.1 150.71) (width 1) (layer "F.Cu") (net 37))
-  (segment (start 159.2 83.79) (end 158.22 82.81) (width 1) (layer "F.Cu") (net 37))
   (segment (start 145.24 86.22) (end 145.25 86.23) (width 0.6) (layer "F.Cu") (net 37))
-  (segment (start 141.171307 164.91) (end 157.3 164.91) (width 1) (layer "F.Cu") (net 37))
-  (segment (start 149.1 86.23) (end 145.25 86.23) (width 1) (layer "F.Cu") (net 37))
+  (segment (start 159.2 83.79) (end 158.22 82.81) (width 1) (layer "F.Cu") (net 37))
   (segment (start 159.05 109.96) (end 159.1 110.01) (width 1) (layer "F.Cu") (net 37))
   (segment (start 146.78 153.78) (end 149.98 150.58) (width 1) (layer "F.Cu") (net 37))
+  (segment (start 158.22 82.81) (end 152.52 82.81) (width 1) (layer "F.Cu") (net 37))
   (segment (start 143.62 86.22) (end 145.24 86.22) (width 0.6) (layer "F.Cu") (net 37))
   (segment (start 147.13 126.76) (end 150.17 123.72) (width 1) (layer "F.Cu") (net 37))
@@
   (segment (start 145.25 153.8) (end 145.27 153.78) (width 0.5) (layer "F.Cu") (net 37))
   (segment (start 159.03 137.14) (end 159.1 137.21) (width 1) (layer "F.Cu") (net 37))
-  (segment (start 123.41 147.148693) (end 141.171307 164.91) (width 1) (layer "F.Cu") (net 37))
   (segment (start 159.1 96.28) (end 150.41 96.28) (width 1) (layer "F.Cu") (net 37))
   (segment (start 145.52 140.26) (end 146.56 140.26) (width 1) (layer "F.Cu") (net 37))
-  (segment (start 158.22 82.81) (end 152.52 82.81) (width 1) (layer "F.Cu") (net 37))
   (segment (start 150.49 109.96) (end 159.05 109.96) (width 1) (layer "F.Cu") (net 37))
   (segment (start 150.17 123.72) (end 159.01 123.72) (width 1) (layer "F.Cu") (net 37))
   (segment (start 143.73 153.8) (end 145.25 153.8) (width 0.6) (layer "F.Cu") (net 37))
+  (segment (start 123.5 164.91) (end 157.3 164.91) (width 1) (layer "F.Cu") (net 37))
   (segment (start 146.56 140.26) (end 149.68 137.14) (width 1) (layer "F.Cu") (net 37))
   (segment (start 143.7 126.76) (end 145.26 126.76) (width 0.6) (layer "F.Cu") (net 37))
+  (segment (start 157.3 164.91) (end 159.2 163.01) (width 1) (layer "F.Cu") (net 37))
   (segment (start 145.51 140.25) (end 145.52 140.26) (width 0.5) (layer "F.Cu") (net 37))
-  (segment (start 123.41 146.035) (end 123.41 147.148693) (width 1) (layer "F.Cu") (net 37))
+  (segment (start 159.2 163.01) (end 159.2 83.79) (width 1) (layer "F.Cu") (net 37))
   (segment (start 147.16 113.29) (end 150.49 109.96) (width 1) (layer "F.Cu") (net 37))
-  (segment (start 157.3 164.91) (end 159.2 163.01) (width 1) (layer "F.Cu") (net 37))
+  (segment (start 152.52 82.81) (end 149.1 86.23) (width 1) (layer "F.Cu") (net 37))
+  (segment (start 123.41 164.82) (end 123.5 164.91) (width 1) (layer "F.Cu") (net 37))
   (segment (start 145.26 126.76) (end 147.13 126.76) (width 1) (layer "F.Cu") (net 37))
   (segment (start 150.41 96.28) (end 147 99.69) (width 1) (layer "F.Cu") (net 37))
@@
   (segment (start 145.27 153.78) (end 146.78 153.78) (width 1) (layer "F.Cu") (net 37))
   (segment (start 143.67 113.25) (end 145.15 113.25) (width 0.6) (layer "F.Cu") (net 37))
-  (segment (start 152.52 82.81) (end 149.1 86.23) (width 1) (layer "F.Cu") (net 37))
   (segment (start 110.4425 108.4575) (end 110.4425 108.41) (width 0.25) (layer "F.Cu") (net 44))
   (segment (start 104.26 112.67) (end 103.285 112.67) (width 0.25) (layer "F.Cu") (net 44))
