File: Harpe ruches/Fichier Kicad/Harpe_ESP32/TestboardV2.3a.kicad_sch (KiCad schematic)
At the start: 15 parts, among them J1 Conn_01x04, J10 Screw_Terminal_01x02, J7 Conn_01x04, Q2 DMG2301L, U13 XC6220B331MR

Commit message: Update PCB
Parts:
- removed J10: Screw_Terminal_01x02, Empreintes:1190297, symbol Connector:Screw_Terminal_01x02
- added J8: Conn_01x04, Empreintes:1190297, symbol Connector_Generic:Conn_01x04
Connections:
- net GND: now also J8.1 (Pin_1), J8.2 (Pin_2)
- net VBAT: now also J8.3 (Pin_3), J8.4 (Pin_4)
Changed lines of the file:
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@@
   (junction (at 173.99 137.668) (diameter 0) (color 0 0 0 0)
   )
+  (junction (at 82.296 146.558) (diameter 0) (color 0 0 0 0)
+  )
   (junction (at 232.41 140.208) (diameter 0) (color 0 0 0 0)
   )
   (junction (at 243.84 140.208) (diameter 0) (color 0 0 0 0)
   )
+  (junction (at 80.772 141.478) (diameter 0) (color 0 0 0 0)
+  )
   (junction (at 52.578 34.29) (diameter 0) (color 0 0 0 0)
   )
@@
     (stroke (width 0) (type default))
   )
+  (wire (pts (xy 67.31 141.478) (xy 67.31 146.558))
+    (stroke (width 0) (type default))
+  )
   (wire (pts (xy 217.17 39.878) (xy 217.17 46.228))
     (stroke (width 0) (type default))
@@
     (stroke (width 0) (type default))
   )
+  (wire (pts (xy 80.772 141.478) (xy 67.31 141.478))
+    (stroke (width 0) (type default))
+  )
   (wire (pts (xy 232.41 141.478) (xy 232.41 140.208))
     (stroke (width 0) (type default))
@@
     (stroke (width 0) (type default))
   )
+  (wire (pts (xy 83.566 141.478) (xy 80.772 141.478))
+    (stroke (width 0) (type default))
+  )
   (wire (pts (xy 184.15 137.668) (xy 184.15 141.478))
     (stroke (width 0) (type default))
@@
     (stroke (width 0) (type default))
   )
+  (wire (pts (xy 80.772 146.558) (xy 82.296 146.558))
+    (stroke (width 0) (type default))
+  )
   (wire (pts (xy 72.136 69.088) (xy 72.136 72.898))
     (stroke (width 0) (type default))
@@
     (stroke (width 0) (type default))
   )
-  (wire (pts (xy 61.468 130.302) (xy 76.2 130.302))
-    (stroke (width 0) (type default))
-  )
   (wire (pts (xy 236.982 90.932) (xy 231.902 90.932))
     (stroke (width 0) (type default))
@@
     (stroke (width 0) (type default))
   )
-  (wire (pts (xy 61.468 130.302) (xy 61.468 134.112))
-    (stroke (width 0) (type default))
-  )
   (wire (pts (xy 201.93 150.368) (xy 215.9 150.368))
     (stroke (width 0) (type default))
@@
     (stroke (width 0) (type default))
   )
+  (wire (pts (xy 80.772 141.478) (xy 80.772 144.018))
+    (stroke (width 0) (type default))
+  )
   (wire (pts (xy 76.2 86.36) (xy 66.04 86.36))
     (stroke (width 0) (type default))
@@
     (stroke (width 0) (type default))
   )
-  (wire (pts (xy 73.914 132.842) (xy 76.2 132.842))
+  (wire (pts (xy 82.296 146.558) (xy 83.566 146.558))
     (stroke (width 0) (type default))
   )
@@
     (stroke (width 0) (type default))
   )
+  (wire (pts (xy 80.772 144.018) (xy 83.566 144.018))
+    (stroke (width 0) (type default))
+  )
   (wire (pts (xy 55.118 35.56) (xy 52.578 35.56))
     (stroke (width 0) (type default))
@@
     (stroke (width 0) (type default))
   )
+  (wire (pts (xy 82.296 146.558) (xy 82.296 149.098))
+    (stroke (width 0) (type default))
+  )
   (wire (pts (xy 158.75 46.228) (xy 158.75 34.798))
     (stroke (width 0) (type default))
@@
   )
   (wire (pts (xy 201.93 140.208) (xy 201.93 150.368))
+    (stroke (width 0) (type default))
+  )
+  (wire (pts (xy 82.296 149.098) (xy 83.566 149.098))
     (stroke (width 0) (type default))
   )
@@
     (effects (font (size 1.27 1.27)) (justify left bottom))
   )
-  (global_label "VBAT" (shape output) (at 73.914 132.842 180)
-    (effects (font (size 1.27 1.27)) (justify right))
-    (property "Intersheetrefs" "${INTERSHEET_REFS}" (at 73.914 132.842 0)
-      (effects (font (size 1.27 1.27)) hide)
-    )
-  )
   (global_label "+3V3" (shape input) (at 66.04 83.82 180)
     (effects (font (size 1.27 1.27)) (justify right))
@@
     (effects (font (size 1.27 1.27)) (justify right))
     (property "Intersheetrefs" "${INTERSHEET_REFS}" (at 65.786 61.468 0)
+      (effects (font (size 1.27 1.27)) hide)
+    )
+  )
+  (global_label "VBAT" (shape output) (at 80.772 146.558 180)
+    (effects (font (size 1.27 1.27)) (justify right))
+    (property "Intersheetrefs" "${INTERSHEET_REFS}" (at 80.772 146.558 0)
       (effects (font (size 1.27 1.27)) hide)
     )
@@
     )
   )
-  (symbol (lib_id "Connector:Screw_Terminal_01x02") (at 81.28 130.302 0) (unit 1)
-    (in_bom yes) (on_board yes) (dnp no) (fields_autoplaced)
-    (property "Reference" "J10" (at 83.312 130.9283 0)
-      (effects (font (size 1.27 1.27)) (justify left))
-    )
-    (property "Value" "Screw_Terminal_01x02" (at 83.312 132.8493 0)
-      (effects (font (size 1.27 1.27)) (justify left))
-    )
-    (property "Footprint" "Empreintes:1190297" (at 81.28 130.302 0)
-      (effects (font (size 1.27 1.27)) hide)
-    )
-    (property "Datasheet" "~" (at 81.28 130.302 0)
-      (effects (font (size 1.27 1.27)) hide)
-    )
-    (pin "1")
-    (pin "3")
-    (instances
-      (project "Harpe_ESP32"
-        (path "/3d1bb011-3bf9-4cd9-8566-e747d5442684/00000000-0000-0000-0000-00006011445d"
-          (reference "J10") (unit 1)
-        )
-      )
-    )
-  )
   (symbol (lib_id "Device:C") (at 194.31 145.288 0) (unit 1)
     (in_bom yes) (on_board yes) (dnp no)
@@
         (path "/3d1bb011-3bf9-4cd9-8566-e747d5442684/00000000-0000-0000-0000-00006011445d"
           (reference "J1") (unit 1)
+        )
+      )
+    )
+  )
+  (symbol (lib_id "Connector_Generic:Conn_01x04") (at 88.646 144.018 0) (unit 1)
+    (in_bom yes) (on_board yes) (dnp no) (fields_autoplaced)
+    (property "Reference" "J8" (at 90.678 144.6443 0)
+      (effects (font (size 1.27 1.27)) (justify left))
+    )
+    (property "Value" "Conn_01x04" (at 90.678 146.5653 0)
+      (effects (font (size 1.27 1.27)) (justify left))
+    )
+    (property "Footprint" "Empreintes:1190297" (at 88.646 144.018 0)
+      (effects (font (size 1.27 1.27)) hide)
+    )
+    (property "Datasheet" "~" (at 88.646 144.018 0)
+      (effects (font (size 1.27 1.27)) hide)
+    )
+    (pin "1")
+    (pin "2")
+    (pin "3")
+    (pin "4")
+    (instances
+      (project "Harpe_ESP32"
+        (path "/3d1bb011-3bf9-4cd9-8566-e747d5442684"
+          (reference "J8") (unit 1)
+        )
+        (path "/3d1bb011-3bf9-4cd9-8566-e747d5442684/00000000-0000-0000-0000-00006011445d"
+          (reference "J11") (unit 1)
         )
       )
@@
     )
   )
-  (symbol (lib_id "power:GND") (at 61.468 134.112 0) (unit 1)
-    (in_bom yes) (on_board yes) (dnp no)
-    (property "Reference" "#PWR08" (at 61.468 140.462 0)
-      (effects (font (size 1.27 1.27)) hide)
-    )
-    (property "Value" "GND" (at 61.595 138.5062 0)
-      (effects (font (size 1.27 1.27)))
-    )
-    (property "Footprint" "" (at 61.468 134.112 0)
-      (effects (font (size 1.27 1.27)) hide)
-    )
-    (property "Datasheet" "" (at 61.468 134.112 0)
-      (effects (font (size 1.27 1.27)) hide)
-    )
-    (pin "1")
-    (instances
-      (project "Harpe_ESP32"
-        (path "/3d1bb011-3bf9-4cd9-8566-e747d5442684/00000000-0000-0000-0000-00006011445d"
-          (reference "#PWR08") (unit 1)
-        )
-      )
-    )
-  )
   (symbol (lib_id "power:GND") (at 232.41 152.908 0) (unit 1)
     (in_bom yes) (on_board yes) (dnp no)
@@
         )
       )
+    )
+  )
+  (symbol (lib_id "power:GND") (at 67.31 146.558 0) (unit 1)
+    (in_bom yes) (on_board yes) (dnp no)
+    (property "Reference" "#PWR014" (at 67.31 152.908 0)
+      (effects (font (size 1.27 1.27)) hide)
+    )
+    (property "Value" "GND" (at 67.437 150.9522 0)
+      (effects (font (size 1.27 1.27)) hide)
+    )
+    (property "Footprint" "" (at 67.31 146.558 0)
+      (effects (font (size 1.27 1.27)) hide)
+    )
+    (property "Datasheet" "" (at 67.31 146.558 0)
+      (effects (font (size 1.27 1.27)) hide)
+    )
+    (pin "1")
+    (instances
+      (project "Harpe_ESP32"
+        (path "/3d1bb011-3bf9-4cd9-8566-e747d5442684"
+          (reference "#PWR014") (unit 1)
+        )
+        (path "/3d1bb011-3bf9-4cd9-8566-e747d5442684/00000000-0000-0000-0000-00006011445d"
+          (reference "#PWR017") (unit 1)
+        )
+      )

Commit message: update
Parts:
- J8: footprint Empreintes:1190297 -> Empreintes:1862411
Changed lines of the file:
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@@
       (effects (font (size 1.27 1.27)) (justify left))
     )
-    (property "Footprint" "Empreintes:1190297" (at 88.646 144.018 0)
+    (property "Footprint" "Empreintes:1862411" (at 88.646 144.018 0)
       (effects (font (size 1.27 1.27)) hide)
     )

Commit message: update
Other:
- title: TestboardV2.3a -> Harpes_ESP32a
Changed lines of the file:
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@@
   (paper "A4")
   (title_block
-    (title "TestboardV2.3a")
+    (title "Harpes_ESP32a")
     (date "2021-12-11")
   )
