File: Harpe ruches/Fichier Kicad/Harpe_ESP32/TestboardV2.3b.kicad_sch (KiCad schematic)
At the start: 0 parts

Commit message: update
Other:
- title: Testboard V2.3b -> Harpes_ESP32b
Changed lines of the file:
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@@
   (paper "A4")
   (title_block
-    (title "Testboard V2.3b")
+    (title "Harpes_ESP32b")
     (date "2021-12-11")
   )
