File: Harpe ruches/Fichier Kicad/Harpe_ESP32/_autosave-Harpe_ESP32.kicad_pcb (KiCad board)
At the start: 2 copper layers, 69.3 x 100 mm, 69 parts, among them J1 Conn_01x04, J10 Conn_01x02, J11 Conn_01x04, J13 USB_C_Receptacle_USB2.0 USB41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, J2 Conn_01x04, J3 Conn_01x04, J4 Conn_01x04, J5 Conn_01x04, J6 Conn_01x04, J7 Conn_01x04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

Commit message: update
Parts:
- moved REF** 3.89 mm to (107.2, 89.1)
- moved REF** 3.65 mm to (100.8, 88.9)
- moved G*** 1.37 mm to (127.8, 103.1)
Changed lines of the file:
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@@
   )
   (footprint "Symbol:OSHW-Logo2_7.3x6mm_SilkScreen" (layer "B.Cu")
-    (at 108.87 92.64 180)
+    (at 107.21 89.12 180)
     (descr "Open Source Hardware Symbol")
     (tags "Logo Symbol OSHW")
@@
   )
   (footprint "Symbol:WEEE-Logo_4.2x6mm_SilkScreen" (layer "B.Cu")
-    (at 102.27 92.27 180)
+    (at 100.84 88.91 180)
     (descr "Waste Electrical and Electronic Equipment Directive")
     (tags "Logo WEEE")
@@
   )
   (footprint "Empreintes:logo frelon" (layer "B.Cu")
-    (at 129.14 103.12 180)
+    (at 127.77 103.09 180)
     (attr board_only exclude_from_pos_files exclude_from_bom)
     (fp_text reference "G***" (at 0 0) (layer "B.SilkS") hide
@@
     (effects (font (size 1 1) (thickness 0.2) bold) (justify mirror))
   )
-  (gr_text "By Ratamuse" (at 111.5 165.34) (layer "B.SilkS")
+  (gr_text "By Ratamuse" (at 109.78 165.34) (layer "B.SilkS")
     (effects (font (size 1.5 1.5) (thickness 0.3)) (justify mirror))
   )
