File: Harpe ruches/Fichier Kicad/Harpe_ESP32/Harpe_ESP32.kicad_sch (KiCad schematic)
At the start: 42 parts, among them J13 USB_C_Receptacle_USB2.0 USB41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, J2 Conn_01x02_MountingPin, J3 Conn_01x02_MountingPin, J4 Conn_01x02_MountingPin, J5 Conn_01x02_MountingPin, J6 Conn_01x02_MountingPin, J8 Conn_01x02_MountingPin, Q1 UMH3N, SW1 SW_Push, U1 ESP32-WROOM-32D, U12 CP2102N-A02-GQFN24, U2 PC817, U3 PC817, U4 PC817, U5 PC817, U6 PC817, U7 PC817

Commit message: Update PCB
Parts:
- added J9: Conn_01x02, symbol Connector_Generic:Conn_01x02
- added R8: 10K, Resistor_SMD:R_0603_1608Metric, symbol Device:R
- added SW2: SW_Push, Empreintes:PTS636SL43SMTRLFS, symbol Switch:SW_Push
Connections:
- net +3V3: now also R8.2
- net GND: now also J9.1 (Pin_1), SW2.2
- net I012: now reaches U1.14 (IO12)
- net I012: now also J9.2 (Pin_2), R8.1, SW2.1
Changed lines of the file:
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@@
   (junction (at 193.04 55.88) (diameter 0) (color 0 0 0 0)
   )
+  (junction (at 158.242 146.558) (diameter 0) (color 0 0 0 0)
+  )
   (junction (at 38.1 109.22) (diameter 0) (color 0 0 0 0)
   )
@@
   (junction (at 38.1 85.09) (diameter 0) (color 0 0 0 0)
   )
+  (junction (at 141.224 146.558) (diameter 0) (color 0 0 0 0)
+  )
   (junction (at 69.85 35.56) (diameter 0) (color 0 0 0 0)
   )
@@
   (junction (at 52.07 27.94) (diameter 0) (color 0 0 0 0)
   )
+  (junction (at 146.05 146.558) (diameter 0) (color 0 0 0 0)
+  )
   (junction (at 46.99 109.22) (diameter 0) (color 0 0 0 0)
   )
@@
     (stroke (width 0) (type default))
   )
+  (wire (pts (xy 153.924 156.972) (xy 153.924 151.892))
+    (stroke (width 0) (type default))
+  )
+  (wire (pts (xy 171.958 146.558) (xy 171.958 151.638))
+    (stroke (width 0) (type default))
+  )
   (wire (pts (xy 215.9 19.05) (xy 215.9 48.26))
     (stroke (width 0) (type default))
@@
     (stroke (width 0) (type default))
   )
+  (wire (pts (xy 137.668 146.558) (xy 141.224 146.558))
+    (stroke (width 0) (type default))
+  )
   (wire (pts (xy 245.11 19.05) (xy 219.71 19.05))
     (stroke (width 0) (type default))
@@
     (stroke (width 0) (type default))
   )
+  (wire (pts (xy 158.242 151.892) (xy 158.242 146.558))
+    (stroke (width 0) (type default))
+  )
   (wire (pts (xy 134.62 88.9) (xy 132.08 88.9))
     (stroke (width 0) (type default))
@@
     (stroke (width 0) (type default))
   )
+  (wire (pts (xy 82.55 124.46) (xy 87.63 124.46))
+    (stroke (width 0) (type default))
+  )
   (wire (pts (xy 59.69 17.78) (xy 54.61 17.78))
     (stroke (width 0) (type default))
@@
     (stroke (width 0) (type default))
   )
+  (wire (pts (xy 146.05 146.558) (xy 146.558 146.558))
+    (stroke (width 0) (type default))
+  )
   (wire (pts (xy 69.85 59.69) (xy 69.85 66.04))
     (stroke (width 0) (type default))
@@
     (stroke (width 0) (type default))
   )
+  (wire (pts (xy 151.384 151.892) (xy 151.384 156.972))
+    (stroke (width 0) (type default))
+  )
   (wire (pts (xy 82.55 134.62) (xy 87.63 134.62))
     (stroke (width 0) (type default))
@@
     (stroke (width 0) (type default))
   )
+  (wire (pts (xy 151.384 151.892) (xy 146.05 151.892))
+    (stroke (width 0) (type default))
+  )
   (wire (pts (xy 125.73 81.28) (xy 134.874 81.28))
     (stroke (width 0) (type default))
@@
     (stroke (width 0) (type default))
   )
+  (wire (pts (xy 156.718 146.558) (xy 158.242 146.558))
+    (stroke (width 0) (type default))
+  )
   (wire (pts (xy 107.95 86.36) (xy 107.95 88.9))
     (stroke (width 0) (type default))
@@
     (stroke (width 0) (type default))
   )
+  (wire (pts (xy 146.05 151.892) (xy 146.05 146.558))
+    (stroke (width 0) (type default))
+  )
   (wire (pts (xy 30.48 85.09) (xy 38.1 85.09))
     (stroke (width 0) (type default))
@@
     (stroke (width 0) (type default))
   )
+  (wire (pts (xy 153.924 151.892) (xy 158.242 151.892))
+    (stroke (width 0) (type default))
+  )
   (wire (pts (xy 52.07 116.84) (xy 49.53 116.84))
     (stroke (width 0) (type default))
@@
     (stroke (width 0) (type default))
   )
+  (wire (pts (xy 141.224 146.558) (xy 141.224 153.67))
+    (stroke (width 0) (type default))
+  )
   (wire (pts (xy 38.1 40.64) (xy 41.91 40.64))
     (stroke (width 0) (type default))
@@
     (stroke (width 0) (type default))
   )
+  (wire (pts (xy 141.224 146.558) (xy 146.05 146.558))
+    (stroke (width 0) (type default))
+  )
   (wire (pts (xy 107.95 49.53) (xy 107.95 52.07))
     (stroke (width 0) (type default))
@@
     (stroke (width 0) (type default))
   )
+  (wire (pts (xy 158.242 146.558) (xy 171.958 146.558))
+    (stroke (width 0) (type default))
+  )
   (wire (pts (xy 134.62 49.53) (xy 125.73 49.53))
     (stroke (width 0) (type default))
@@
     (stroke (width 0) (type default))
   )
+  (wire (pts (xy 125.73 146.558) (xy 130.048 146.558))
+    (stroke (width 0) (type default))
+  )
   (wire (pts (xy 134.62 52.07) (xy 132.08 52.07))
     (stroke (width 0) (type default))
@@
     (effects (font (size 1.27 1.27)) (justify left))
     (property "Intersheetrefs" "${INTERSHEET_REFS}" (at 87.63 142.24 0)
+      (effects (font (size 1.27 1.27)) hide)
+    )
+  )
+  (global_label "+3V3" (shape input) (at 125.73 146.558 180)
+    (effects (font (size 1.27 1.27)) (justify right))
+    (property "Intersheetrefs" "${INTERSHEET_REFS}" (at 125.73 146.558 0)
       (effects (font (size 1.27 1.27)) hide)
     )
@@
     )
   )
+  (global_label "I012" (shape output) (at 141.224 153.67 270)
+    (effects (font (size 1.27 1.27)) (justify right))
+    (property "Intersheetrefs" "${INTERSHEET_REFS}" (at 141.224 153.67 0)
+      (effects (font (size 1.27 1.27)) hide)
+    )
+  )
   (global_label "RTS" (shape input) (at 247.65 86.36 180)
     (effects (font (size 1.27 1.27)) (justify right))
@@
     (effects (font (size 1.27 1.27)) (justify right))
     (property "Intersheetrefs" "${INTERSHEET_REFS}" (at 208.28 60.96 0)
+      (effects (font (size 1.27 1.27)) hide)
+    )
+  )
+  (global_label "I012" (shape input) (at 87.63 124.46 0)
+    (effects (font (size 1.27 1.27)) (justify left))
+    (property "Intersheetrefs" "${INTERSHEET_REFS}" (at 87.63 124.46 0)
       (effects (font (size 1.27 1.27)) hide)
     )
@@
     )
   )
+  (symbol (lib_id "Connector_Generic:Conn_01x02") (at 153.924 162.052 270) (unit 1)
+    (in_bom yes) (on_board yes) (dnp no) (fields_autoplaced)
+    (property "Reference" "J9" (at 155.956 161.4083 90)
+      (effects (font (size 1.27 1.27)) (justify left))
+    )
+    (property "Value" "Conn_01x02" (at 155.956 163.3293 90)
+      (effects (font (size 1.27 1.27)) (justify left))
+    )
+    (property "Footprint" "" (at 153.924 162.052 0)
+      (effects (font (size 1.27 1.27)) hide)
+    )
+    (property "Datasheet" "~" (at 153.924 162.052 0)
+      (effects (font (size 1.27 1.27)) hide)
+    )
+    (pin "1")
+    (pin "2")
+    (instances
+      (project "Harpe_ESP32"
+        (path "/3d1bb011-3bf9-4cd9-8566-e747d5442684"
+          (reference "J9") (unit 1)
+        )
+      )
+    )
+  )
   (symbol (lib_id "power:GND") (at 132.08 91.44 0) (unit 1)
     (in_bom yes) (on_board yes) (dnp no)
@@
     )
   )
+  (symbol (lib_id "Device:R") (at 133.858 146.558 270) (unit 1)
+    (in_bom yes) (on_board yes) (dnp no)
+    (property "Reference" "R8" (at 133.858 141.3002 90)
+      (effects (font (size 1.27 1.27)))
+    )
+    (property "Value" "10K" (at 133.858 143.6116 90)
+      (effects (font (size 1.27 1.27)))
+    )
+    (property "Footprint" "Resistor_SMD:R_0603_1608Metric" (at 133.858 144.78 90)
+      (effects (font (size 1.27 1.27)) hide)
+    )
+    (property "Datasheet" "~" (at 133.858 146.558 0)
+      (effects (font (size 1.27 1.27)) hide)
+    )
+    (pin "1")
+    (pin "2")
+    (instances
+      (project "Harpe_ESP32"
+        (path "/3d1bb011-3bf9-4cd9-8566-e747d5442684"
+          (reference "R8") (unit 1)
+        )
+      )
+    )
+  )
+  (symbol (lib_id "power:GND") (at 171.958 151.638 0) (unit 1)
+    (in_bom yes) (on_board yes) (dnp no)
+    (property "Reference" "#PWR015" (at 171.958 157.988 0)
+      (effects (font (size 1.27 1.27)) hide)
+    )
+    (property "Value" "GND" (at 172.085 156.0322 0)
+      (effects (font (size 1.27 1.27)))
+    )
+    (property "Footprint" "" (at 171.958 151.638 0)
+      (effects (font (size 1.27 1.27)) hide)
+    )
+    (property "Datasheet" "" (at 171.958 151.638 0)
+      (effects (font (size 1.27 1.27)) hide)
+    )
+    (pin "1")
+    (instances
+      (project "Harpe_ESP32"
+        (path "/3d1bb011-3bf9-4cd9-8566-e747d5442684"
+          (reference "#PWR015") (unit 1)
+        )
+      )
+    )
+  )
   (symbol (lib_id "power:GND") (at 132.08 34.29 0) (unit 1)
     (in_bom yes) (on_board yes) (dnp no)
@@
         )
       )
+    )
+  )
+  (symbol (lib_id "Switch:SW_Push") (at 151.638 146.558 0) (unit 1)
+    (in_bom yes) (on_board yes) (dnp no)
+    (property "Reference" "SW2" (at 151.638 139.319 0)
+      (effects (font (size 1.27 1.27)))
+    )
+    (property "Value" "SW_Push" (at 151.638 141.6304 0)
+      (effects (font (size 1.27 1.27)))
+    )
+    (property "Footprint" "Empreintes:PTS636SL43SMTRLFS" (at 151.638 141.478 0)
+      (effects (font (size 1.27 1.27)) hide)
+    )
+    (property "Datasheet" "~" (at 151.638 141.478 0)
+      (effects (font (size 1.27 1.27)) hide)
+    )
+    (pin "1")
+    (pin "2")
+    (instances
+      (project "Harpe_ESP32"
+        (path "/3d1bb011-3bf9-4cd9-8566-e747d5442684"
+          (reference "SW2") (unit 1)
+        )
+      )

Commit message: Update PCB
Parts:
- removed J2, J3, J4, J5, J6, J8: Conn_01x02_MountingPin, Empreintes:1190297, symbol Connector:Screw_Terminal_01x02
- added J10: Conn_01x02, Connector_JST:JST_PH_B2B-PH-K_1x02_P2.00mm_Vertical, symbol Connector_Generic:Conn_01x02
- added J2, J3, J4, J5, J6, J8: Conn_01x04, Empreintes:1190297, symbol Connector_Generic:Conn_01x04
- J9: footprint (none) -> Connector_JST:JST_PH_B2B-PH-K_1x02_P2.00mm_Vertical
Connections:
- net GND: now also J9.2 (Pin_2), J10.2 (Pin_2), J2.3 (Pin_3), J2.4 (Pin_4), J3.3 (Pin_3), J3.4 (Pin_4), J4.3 (Pin_3), J4.4 (Pin_4), J5.3 (Pin_3), J5.4 (Pin_4), J6.3 (Pin_3), J6.4 (Pin_4), J8.3 (Pin_3), J8.4 (Pin_4); no longer J9.1 (Pin_1)
- net RST_EN: now also J10.1 (Pin_1)
- net I027: now reaches U1.12 (IO27)
- net I027: now also J9.1 (Pin_1), R8.1, SW2.1
- net I023: now reaches U1.37 (IO23)
- net at U5.3: now also J5.1 (Pin_1), J5.2 (Pin_2)
- net at U6.3: now also J6.1 (Pin_1), J6.2 (Pin_2)
- net at U7.3: now also J8.1 (Pin_1), J8.2 (Pin_2)
- net at U2.3: now also J2.1 (Pin_1), J2.2 (Pin_2)
- net at U3.3: now also J3.1 (Pin_1), J3.2 (Pin_2)
- removed net I012: J9.2 (Pin_2), R8.1, SW2.1, U1.14 (IO12)
- new net: J4.1 (Pin_1), J4.2 (Pin_2)
Other:
- moved on the sheet: J9

Commit message: update
Parts:
- J2, J3, J4, J5, J6, J8: footprint Empreintes:1190297 -> Empreintes:1862411
Connections:
- net at U4.3: now also J4.1 (Pin_1), J4.2 (Pin_2)
Changed lines of the file:
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@@
-    (stroke (width 0) (type default))
-  )
-  (wire (pts (xy 132.08 68.58) (xy 125.984 68.58))
     (stroke (width 0) (type default))
   )
@@
   )
   (wire (pts (xy 149.86 109.22) (xy 149.86 111.76))
+    (stroke (width 0) (type default))
+  )
+  (wire (pts (xy 125.73 68.58) (xy 132.08 68.58))
     (stroke (width 0) (type default))
   )
@@
       (effects (font (size 1.27 1.27)) (justify left))
     )
-    (property "Footprint" "Empreintes:1190297" (at 156.21 123.19 0)
+    (property "Footprint" "Empreintes:1862411" (at 156.21 123.19 0)
       (effects (font (size 1.27 1.27)) hide)
     )
@@
       (effects (font (size 1.27 1.27)) (justify left))
     )
-    (property "Footprint" "Empreintes:1190297" (at 156.21 106.68 0)
+    (property "Footprint" "Empreintes:1862411" (at 156.21 106.68 0)
       (effects (font (size 1.27 1.27)) hide)
     )
@@
       (effects (font (size 1.27 1.27)) (justify left))
     )
-    (property "Footprint" "Empreintes:1190297" (at 139.7 31.75 0)
+    (property "Footprint" "Empreintes:1862411" (at 139.7 31.75 0)
       (effects (font (size 1.27 1.27)) hide)
     )
@@
       (effects (font (size 1.27 1.27)) (justify left))
     )
-    (property "Footprint" "Empreintes:1190297" (at 139.7 88.9 0)
+    (property "Footprint" "Empreintes:1862411" (at 139.7 88.9 0)
       (effects (font (size 1.27 1.27)) hide)
     )
@@
       (effects (font (size 1.27 1.27)) (justify left))
     )
-    (property "Footprint" "Empreintes:1190297" (at 139.954 71.12 0)
+    (property "Footprint" "Empreintes:1862411" (at 139.954 71.12 0)
       (effects (font (size 1.27 1.27)) hide)
     )
@@
       (effects (font (size 1.27 1.27)) (justify left))
     )
-    (property "Footprint" "Empreintes:1190297" (at 139.7 52.07 0)
-      (effects (font (size 1.27 1.27)) hide)
-    )
+    (property "Footprint" "Empreintes:1862411" (at 139.7 52.07 0)
+      (effects (font (size 1.27 1.27)) hide)
+    )

Commit message: update
Parts:
- U2, U3, U4, U5, U6, U7: value PC817 -> G3VM-61VY2; footprint Empreintes:SOP254P960X420-4N -> Empreintes:SOP254P700X230-4N
Other:
- moved on the sheet: J6, J8, R6, R7
