File: Harpe ruches/Fichier Kicad/Harpe_PCB_4_couches/Harpe_PCB_4_couches.kicad_pcb (KiCad board)
At the start: 4 copper layers, 600 x 36.2 mm, 42 parts

Commit message: update
Parts:
- removed the REF** at (39.7, 40.2)
- added ?: , , F.Cu at (40.0, 40.1)
- moved G*** 3.87 mm to (329.4, 50.7)
- moved G*** 3.16 mm to (337.8, 50.9)
Routing:
- net (no net): track 1649.8 -> 1631.0 mm
Other:
- board text added: "Harpe électrique destinée à foudroyer les frelons asiatiques V0.3"
- board text added: "Ratamuse 09/2024"
- board text removed: "Harpe électrique destinée à foudroyer les frelons asiatiques V0.2"
- board text removed: "Ratamuse 05/2024"
